File: audio_interface/audio_interface.kicad_sch (KiCad schematic)
At the start: 57 parts, among them J1 XLR3, J2 AudioJack2, U1 OPA2134, U2 OPA2134, U3 OPA2134, U4 OPA2134

Commit message: Fixed some footprints, fixed silkscreen.
Parts:
- TP1, TP2, TP3, TP4, TP5, TP6, TP7: footprint TestPoint:TestPoint_Loop_D2.54mm_Drill1.5mm_Beaded -> TestPoint:TestPoint_Loop_D2.50mm_Drill1.0mm
Changed lines of the file:
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@@
       (effects (font (size 1.27 1.27)) (justify left))
     )
-    (property "Footprint" "TestPoint:TestPoint_Loop_D2.54mm_Drill1.5mm_Beaded" (id 2) (at 151.13 78.74 0)
+    (property "Footprint" "TestPoint:TestPoint_Loop_D2.50mm_Drill1.0mm" (id 2) (at 151.13 78.74 0)
       (effects (font (size 1.27 1.27)) hide)
     )
@@
       (effects (font (size 1.27 1.27)) (justify left))
     )
-    (property "Footprint" "TestPoint:TestPoint_Loop_D2.54mm_Drill1.5mm_Beaded" (id 2) (at 106.68 156.21 0)
+    (property "Footprint" "TestPoint:TestPoint_Loop_D2.50mm_Drill1.0mm" (id 2) (at 106.68 156.21 0)
       (effects (font (size 1.27 1.27)) hide)
     )
@@
       (effects (font (size 1.27 1.27)) (justify left))
     )
-    (property "Footprint" "TestPoint:TestPoint_Loop_D2.54mm_Drill1.5mm_Beaded" (id 2) (at 259.08 39.37 0)
+    (property "Footprint" "TestPoint:TestPoint_Loop_D2.50mm_Drill1.0mm" (id 2) (at 259.08 39.37 0)
       (effects (font (size 1.27 1.27)) hide)
     )
@@
       (effects (font (size 1.27 1.27)) (justify right))
     )
-    (property "Footprint" "TestPoint:TestPoint_Loop_D2.54mm_Drill1.5mm_Beaded" (id 2) (at 88.9 66.04 0)
+    (property "Footprint" "TestPoint:TestPoint_Loop_D2.50mm_Drill1.0mm" (id 2) (at 88.9 66.04 0)
       (effects (font (size 1.27 1.27)) hide)
     )
@@
       (effects (font (size 1.27 1.27)) (justify right))
     )
-    (property "Footprint" "TestPoint:TestPoint_Loop_D2.54mm_Drill1.5mm_Beaded" (id 2) (at 149.86 171.45 0)
+    (property "Footprint" "TestPoint:TestPoint_Loop_D2.50mm_Drill1.0mm" (id 2) (at 149.86 171.45 0)
       (effects (font (size 1.27 1.27)) hide)
     )
@@
       (effects (font (size 1.27 1.27)) (justify left))
     )
-    (property "Footprint" "TestPoint:TestPoint_Loop_D2.54mm_Drill1.5mm_Beaded" (id 2) (at 259.08 63.5 0)
+    (property "Footprint" "TestPoint:TestPoint_Loop_D2.50mm_Drill1.0mm" (id 2) (at 259.08 63.5 0)
       (effects (font (size 1.27 1.27)) hide)
     )
@@
       (effects (font (size 1.27 1.27)) (justify left))
     )
-    (property "Footprint" "TestPoint:TestPoint_Loop_D2.54mm_Drill1.5mm_Beaded" (id 2) (at 200.66 78.74 0)
+    (property "Footprint" "TestPoint:TestPoint_Loop_D2.50mm_Drill1.0mm" (id 2) (at 200.66 78.74 0)
       (effects (font (size 1.27 1.27)) hide)
     )
@@
     )
     (path "/a848ccfc-ed5a-4abb-b243-1d477e4499b6/9bda60cc-a821-4b43-9290-9cbd01d4101f"
-      (reference "J3") (unit 1) (value "EXT_9V") (footprint "Connector_BarrelJack:BarrelJack_CUI_PJ-063AH_Horizontal")
+      (reference "J3") (unit 1) (value "EXT_9V") (footprint "Connector_BarrelJack:BarrelJack_GCT_DCJ200-10-A_Horizontal")
     )
     (path "/a848ccfc-ed5a-4abb-b243-1d477e4499b6/dc568067-7751-401f-84a8-60bd5c3ab826"
@@
       (reference "JP23") (unit 1) (value "HPFD_n") (footprint "Jumper:SolderJumper-3_P1.3mm_Open_RoundedPad1.0x1.5mm_NumberLabels")
     )
+    (path "/a848ccfc-ed5a-4abb-b243-1d477e4499b6/7dbb2fc9-ee7c-4a13-a074-2dbb8ae45f20"
+      (reference "JP24") (unit 1) (value "Jumper_2_Bridged") (footprint "Resistor_SMD:R_1206_3216Metric_Pad1.30x1.75mm_HandSolder")
+    )
     (path "/92aa0299-bc2d-4ffe-b831-357ccd9e90d2/00aefffa-7d6f-45ca-91c8-39c222a6f0e9"
       (reference "JP27") (unit 1) (value "Jumper_2_Bridged") (footprint "Resistor_SMD:R_1206_3216Metric_Pad1.30x1.75mm_HandSolder")
@@
     )
     (path "/83cfbbe6-d662-44d0-9748-749c34e3a9b6"
-      (reference "TP1") (unit 1) (value "DIFF_OUT_M") (footprint "TestPoint:TestPoint_Loop_D2.54mm_Drill1.5mm_Beaded")
+      (reference "TP1") (unit 1) (value "DIFF_OUT_M") (footprint "TestPoint:TestPoint_Loop_D2.50mm_Drill1.0mm")
     )
     (path "/21487f62-9c22-4ed1-b7e0-fe4a53513e13"
-      (reference "TP2") (unit 1) (value "ADJ_OUT_I") (footprint "TestPoint:TestPoint_Loop_D2.54mm_Drill1.5mm_Beaded")
+      (reference "TP2") (unit 1) (value "ADJ_OUT_I") (footprint "TestPoint:TestPoint_Loop_D2.50mm_Drill1.0mm")
     )
     (path "/058a7166-e51e-486c-9459-32376e832a4f"
-      (reference "TP3") (unit 1) (value "ADJ_OUT_M") (footprint "TestPoint:TestPoint_Loop_D2.54mm_Drill1.5mm_Beaded")
+      (reference "TP3") (unit 1) (value "ADJ_OUT_M") (footprint "TestPoint:TestPoint_Loop_D2.50mm_Drill1.0mm")
     )
     (path "/9704a3e9-5482-47db-8e21-371e5cc974bc"
-      (reference "TP4") (unit 1) (value "BIAS_OUT_I") (footprint "TestPoint:TestPoint_Loop_D2.54mm_Drill1.5mm_Beaded")
+      (reference "TP4") (unit 1) (value "BIAS_OUT_I") (footprint "TestPoint:TestPoint_Loop_D2.50mm_Drill1.0mm")
     )
     (path "/9de977c7-533f-45b9-9358-265f7d3b6076"
-      (reference "TP5") (unit 1) (value "BIAS_OUT_M") (footprint "TestPoint:TestPoint_Loop_D2.54mm_Drill1.5mm_Beaded")
+      (reference "TP5") (unit 1) (value "BIAS_OUT_M") (footprint "TestPoint:TestPoint_Loop_D2.50mm_Drill1.0mm")
     )
     (path "/7f820a05-8bc0-4fdd-a491-41739bf802d8"
-      (reference "TP6") (unit 1) (value "I_BIAS") (footprint "TestPoint:TestPoint_Loop_D2.54mm_Drill1.5mm_Beaded")
+      (reference "TP6") (unit 1) (value "I_BIAS") (footprint "TestPoint:TestPoint_Loop_D2.50mm_Drill1.0mm")
     )
     (path "/9b0622c7-a7c4-468a-a0e2-913087e96668"
-      (reference "TP7") (unit 1) (value "M_BIAS") (footprint "TestPoint:TestPoint_Loop_D2.54mm_Drill1.5mm_Beaded")
+      (reference "TP7") (unit 1) (value "M_BIAS") (footprint "TestPoint:TestPoint_Loop_D2.50mm_Drill1.0mm")
     )
     (path "/a848ccfc-ed5a-4abb-b243-1d477e4499b6/fc734adb-fcad-43e3-aaca-d5f499293016"
-      (reference "TP8") (unit 1) (value "9V") (footprint "TestPoint:TestPoint_Loop_D2.54mm_Drill1.5mm_Beaded")
+      (reference "TP8") (unit 1) (value "9V") (footprint "TestPoint:TestPoint_Loop_D2.50mm_Drill1.0mm")
     )
     (path "/92aa0299-bc2d-4ffe-b831-357ccd9e90d2/ae1e8de8-cf2c-4ad4-8428-bc08c60bb9b8"
@@
     )
     (path "/a848ccfc-ed5a-4abb-b243-1d477e4499b6/e25ee0bf-65fd-4d7b-a3f4-6465bdc4c426"
-      (reference "U7") (unit 1) (value "TPS7A49") (footprint "Package_SO:VSSOP-8_3.0x3.0mm_P0.65mm")
+      (reference "U7") (unit 1) (value "TPS7A49") (footprint "Package_SO:MSOP-8-1EP_3x3mm_P0.65mm_EP1.68x1.88mm_ThermalVias")
     )
     (path "/a848ccfc-ed5a-4abb-b243-1d477e4499b6/c93f38bc-797e-40ff-9143-7684fafc29ad"
-      (reference "U8") (unit 1) (value "TPS7A30") (footprint "Package_SO:VSSOP-8_3.0x3.0mm_P0.65mm")
+      (reference "U8") (unit 1) (value "TPS7A30") (footprint "Package_SO:MSOP-8-1EP_3x3mm_P0.65mm_EP1.68x1.88mm_ThermalVias")
     )
     (path "/a848ccfc-ed5a-4abb-b243-1d477e4499b6/589ea6ea-31af-486b-bfc7-3f9207d8c7e9"
